Commit message: - Updated WAm joint damping and friction based on this (https://www.google.com/url?sa=t&source=web&rct=j&opi=89978449&url=https://figshare.le.ac.uk/articles/The_WAM_arm_modelling_control_and_its_application_in_a_HMI_based_on_gaze_tracking/10165436/files/18320189.pdf&ved=2ahUKEwjL8Mbgg-eKAxUYMNAFHW_pOx4QFnoECBMQAQ&usg=AOvVaw2ZlHKpBFfDdmISZywmNKGY) paper.

File: components/urdf/wam/components_V1.urdf.xacro (robot description, xacro)
@@ -68,6 +68,6 @@
             <origin xyz="0 0 0.346" rpy="0 0 0"/>
             <axis xyz="0 0 1"/>
-            <limit effort="${60}" lower="${-148.97 * M_PI / 180.0}" upper="${148.97 * M_PI / 180.0}" velocity="2.0"/>
-            <dynamics damping="${1.8*b}" friction="0"/>
+            <limit effort="${60}" lower="${-148.97 * M_PI / 180.0}" upper="${148.97 * M_PI / 180.0}" velocity="0.5"/>
+            <dynamics damping="1.3" friction="4.4"/>
         </joint>
         <gazebo reference="${prefix}/J1">
@@ -115,6 +115,6 @@
             <origin xyz="0 0 0" rpy="${-PI/2} 0 0"/>
             <axis xyz="0 0 1"/>
-            <limit effort="${60}" lower="${-113.732 * M_PI / 180.0}" upper="${113.732 * M_PI / 180.0}" velocity="2.0"/>
-            <dynamics damping="${0.5*b}" friction="0"/>
+            <limit effort="${60}" lower="${-113.732 * M_PI / 180.0}" upper="${113.732 * M_PI / 180.0}" velocity="0.5"/>
+            <dynamics damping="3.5" friction="3.5"/>
         </joint>
         <gazebo reference="${prefix}/J2">
@@ -160,6 +160,6 @@
             <origin xyz="0 0 0" rpy="${PI/2} 0 0"/>
             <axis xyz="0 0 1"/>
-            <limit effort="${45}" lower="${-160.428 * M_PI / 180.0}" upper="${160.428 * M_PI / 180.0}" velocity="2.0"/>
-            <dynamics damping="${1.5*b}" friction="0"/>
+            <limit effort="${45}" lower="${-160.428 * M_PI / 180.0}" upper="${160.428 * M_PI / 180.0}" velocity="0.5"/>
+            <dynamics damping="1.2" friction="2.3"/>
         </joint>
         <gazebo reference="${prefix}/J3">
@@ -207,6 +207,6 @@
             <origin xyz="0.045 0 0.55" rpy="${-PI/2} 0 0"/>
             <axis xyz="0 0 1"/>
-            <limit effort="${30}" lower="${-51.567 * M_PI / 180.0}" upper="${180 * M_PI / 180.0}" velocity="2.00"/>
-            <dynamics damping="${0.8*b}" friction="0"/>
+            <limit effort="${30}" lower="${-51.567 * M_PI / 180.0}" upper="${180 * M_PI / 180.0}" velocity="0.50"/>
+            <dynamics damping="2.7" friction="1.5"/>
         </joint>
         <gazebo reference="${prefix}/J4">
@@ -268,6 +268,6 @@
             <origin xyz="-0.045 -0.3 0" rpy="${PI/2} 0 0"/>
             <axis xyz="0 0 1"/>
-            <limit effort="${10}" lower="${-260.696 * M_PI / 180.0}" upper="${71.62 * M_PI / 180.0}" velocity="2.0"/>
-            <dynamics damping="${0.5*b}" friction="0"/>
+            <limit effort="${10}" lower="${-260.696 * M_PI / 180.0}" upper="${71.62 * M_PI / 180.0}" velocity="0.5"/>
+            <dynamics damping="1.46" friction="0.3"/>
         </joint>
         <gazebo reference="${prefix}/J5">
@@ -315,6 +315,6 @@
             <origin xyz="0 0 0" rpy="${-PI/2} 0 0"/>
             <axis xyz="0 0 1"/>
-            <limit effort="${10}" lower="${-90 * M_PI / 180.0}" upper="${90 * M_PI / 180.0}" velocity="2.00"/>
-            <dynamics damping="${0.1*b}" friction="0"/>
+            <limit effort="${10}" lower="${-90 * M_PI / 180.0}" upper="${90 * M_PI / 180.0}" velocity="0.50"/>
+            <dynamics damping="0.8" friction="0.48"/>
         </joint>
         <gazebo reference="${prefix}/J6">
@@ -363,7 +363,7 @@
             <origin xyz="0 0 0" rpy="${PI/2} 0 0"/>
             <axis xyz="0 0 1"/>
-            <limit effort="${10}" lower="${-171.89 * M_PI / 180.0}" upper="${171.89 * M_PI / 180.0}" velocity="2.00"/>
+            <limit effort="${10}" lower="${-171.89 * M_PI / 180.0}" upper="${171.89 * M_PI / 180.0}" velocity="0.50"/>
             <!-- 2.95 is a limit taken in from 3 due to saftey and differences between arms. -->
-            <dynamics damping="${0.1*b}" friction="0"/>
+            <dynamics damping="1" friction="0.13"/>
         </joint>
         <gazebo reference="${prefix}/J7">
@@ -429,5 +429,5 @@
             <limit effort="5" lower="-2.95" upper="2.95" velocity="0.20"/> <!--[> 2.95 is a limit taken in from 3 due to saftey and differences between arms. <]-->
                 <!-- <safety_controller k_position="100" k_velocity="3" soft_lower_limit="-100.0" soft_upper_limit="100.0" /> <] -->
-            <dynamics damping="0.1" friction="100.0"/>
+            <dynamics damping="1" friction="0.13"/>
         </joint>
         <link name="${prefix}/wam_wrist_palm_torque_sensor_link" >
